File: GamesMachine.kicad_sch (KiCad schematic)
At the start: 80 parts, among them IC1 7413, IC10 7480, IC11 7412, IC2 7472, IC3 7490, IC4 7490, IC5 7447, IC6 7447, IC9 7425

Commit message: Fix: tie LOGIC_0 net to GND (schematic side)
LOGIC_0 was drawn as its own local net label, never actually connected
to ground, causing both 7490s to read a floating "1" on their
reset-to-nine inputs and freeze at 99. Renamed all 12 LOGIC_0 labels
to GND, merging it with the existing ground net.

ERC clean of any new conflicts after the change (348 pre-existing
flags, all off-grid/multi-unit-symbol/NC-pin cosmetic categories
unrelated to this net).

PCB side still needs manual attention in Pcbnew: run "Update PCB from
Schematic" and route/zone-fill whatever connections come up unrouted
for the former LOGIC_0 pads (IC2 pins 3/4/5, IC3/IC4 pins 6/7,
S3a/S3b/S5a pin 3, S6c/S6d pin 2) before this is fabrication-ready.

Also adds README and marks decoupling-cap addition as decided against
in the rev 2 fix list.
Connections:
- net LOGIC_0 is gone; now on net GND: IC2.3 (J1), IC2.4 (J2), IC2.5 (J3), IC3.6 (R91), IC3.7 (R92), IC4.6 (R91), IC4.7 (R92), S3a.3 (NO_PRESS), S3b.3 (NO_PRESS), S5a.3 (NO_PRESS), S6c.2 (NC_REL), S6d.2 (NC_REL)
Changed lines of the file:
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@@
 		)
 	)
-	(label "LOGIC_0"
+	(label "GND"
 		(at 131.8 372.76 0)
 		(effects
@@
 		)
 	)
-	(label "LOGIC_0"
+	(label "GND"
 		(at 146.05 142.24 180)
 		(effects
@@
 		)
 	)
-	(label "LOGIC_0"
+	(label "GND"
 		(at 198.92 339.57 0)
 		(effects
@@
 		)
 	)
-	(label "LOGIC_0"
+	(label "GND"
 		(at 248.92 369.57 0)
 		(effects
@@
 		)
 	)
-	(label "LOGIC_0"
+	(label "GND"
 		(at 154.94 281.94 180)
 		(effects
@@
 		)
 	)
-	(label "LOGIC_0"
+	(label "GND"
 		(at 146.05 144.78 180)
 		(effects
@@
 		)
 	)
-	(label "LOGIC_0"
+	(label "GND"
 		(at 154.94 279.4 180)
 		(effects
@@
 		)
 	)
-	(label "LOGIC_0"
+	(label "GND"
 		(at 131.8 332.76 0)
 		(effects
@@
 		)
 	)
-	(label "LOGIC_0"
+	(label "GND"
 		(at 518.87 151.7 0)
 		(effects
@@
 		)
 	)
-	(label "LOGIC_0"
+	(label "GND"
 		(at 46.99 284.48 180)
 		(effects
@@
 		)
 	)
-	(label "LOGIC_0"
+	(label "GND"
 		(at 146.05 139.7 180)
 		(effects
@@
 		)
 	)
-	(label "LOGIC_0"
+	(label "GND"
 		(at 46.99 281.94 180)
 		(effects

Commit message: Fix: diode symbol pin numbering to match stock footprint
The project's cached Device:D symbol had pin 1 = anode, while the
stock DO-35 footprint correctly places the silkscreen cathode band at
pad 1. The footprint was never wrong -- only the schematic's cached
copy of the symbol had drifted from the stock library. Every diode on
rev 1.0 therefore had to be installed opposite the printed band.

Swapped the two pin numbers in the cached symbol (A position now 2,
K position now 1), leaving pin names, graphics and all wiring
untouched. KiCad binds wires by coordinate rather than pin number, so
this corrects all 17 diodes (D5-D20 plus Z1, which share this symbol)
in one edit.

Verified by netlist export: Z1 now pin 1 -> /+5V, pin 2 -> /GND, and
D11 now pin 1 -> /IC3_QA, pin 2 -> /S4A_ROULETTE37 -- both reversed
from before, electrical intent unchanged. ERC unchanged at 348
pre-existing violations with an identical category breakdown.

PCB side still pending: Update PCB from Schematic, verify pad swap,
re-route as needed, and confirm band = cathode on a silkscreen plot.
Connections:
- net +5V: now also Z1.1 (K); no longer Z1.2 (K)
- net GND: now also Z1.2 (A); no longer Z1.1 (A)
- net IC3_QA: now also D11.1 (K), D18.1 (K); no longer D11.2 (K), D18.2 (K)
- net IC3_QB: now also D12.1 (K), D19.1 (K), D9.1 (K); no longer D12.2 (K), D19.2 (K), D9.2 (K)
- net IC3_QC: now also D10.1 (K), D17.1 (K), D20.1 (K); no longer D10.2 (K), D17.2 (K), D20.2 (K)
- net IC4_QA: now also D13.1 (K), D5.1 (K); no longer D13.2 (K), D5.2 (K)
- net IC4_QB: now also D14.1 (K), D6.1 (K); no longer D14.2 (K), D6.2 (K)
- net IC4_QC: now also D15.1 (K), D16.1 (K), D7.1 (K), D8.1 (K); no longer D15.2 (K), D16.2 (K), D7.2 (K), D8.2 (K)
- net S4A_ROULETTE37: now also D11.2 (A), D12.2 (A), D13.2 (A), D14.2 (A), D15.2 (A); no longer D11.1 (A), D12.1 (A), D13.1 (A), D14.1 (A), D15.1 (A)
- net S4B_ROULETTE44: now also D16.2 (A), D17.2 (A); no longer D16.1 (A), D17.1 (A)
- net S5B_POOLS64: now also D10.2 (A), D8.2 (A), D9.2 (A); no longer D10.1 (A), D8.1 (A), D9.1 (A)
- net S6A_DICE_UNITS7: now also D5.2 (A), D6.2 (A), D7.2 (A); no longer D5.1 (A), D6.1 (A), D7.1 (A)
- net S6B_DICE_TENS7: now also D18.2 (A), D19.2 (A), D20.2 (A); no longer D18.1 (A), D19.1 (A), D20.1 (A)

Commit message: Fix: 2N2926 symbol pin order to match the real device (TR1-TR3)
The project-local 2N2926 symbol declared its pins as E-B-C, but the real
2N2926 is E-C-B. That mismatch is why TR1, TR2 and TR3 all had to be
fitted with leads 2 and 3 crossed on the rev 1.0 board.

Swapped the B and C pin numbers in both the source library and the
schematic's cached copy of the symbol. Pin names, positions and graphics
are untouched -- only which pad each pin maps to. Netlist now gives
pad 1 = E, pad 2 = C, pad 3 = B, so the part drops straight into the
TO-92 footprint.

TR4 (2N2646, TO-18) left as is -- confirmed correct as built.

PCB side pending: Update PCB from Schematic, then re-route TR1-TR3,
whose pads 2 and 3 now carry swapped nets.
Parts:
- renumbered PWR to PWR1, S3a to S3a1, S3b to S3b1, S4a to S4a1, S4b to S4b1, S5a to S5a1, S5b to S5b1, S5c to S5c1, S6a to S6a1, S6b to S6b1, S6c to S6c1, S6d to S6d1, TENS to TENS1, UNITS to UNITS1
Connections:
- net N_TR12_BASE: now also TR1.3 (B), TR2.3 (B); no longer TR1.2 (B), TR2.2 (B)
- net N_TR2C: now also TR2.2 (C); no longer TR2.3 (C)
- net N_TR3B: now also TR3.3 (B); no longer TR3.2 (B)
- net N_TR3C: now also TR3.2 (C); no longer TR3.3 (C)
Changed lines of the file:
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@@
 		(on_board yes)
 		(dnp no)
-		(property "Reference" "S6b"
+		(property "Reference" "S6b1"
 			(at 513.79 196.31 0)
 			(effects
@@
 			(project "GamesMachine"
 				(path "/8b2932eb-08c7-412c-8772-7207c8d67aa1"
-					(reference "S6b")
+					(reference "S6b1")
 					(unit 1)
 				)
@@
 		(on_board yes)
 		(dnp no)
-		(property "Reference" "S5c"
+		(property "Reference" "S5c1"
 			(at 187.49 365.61 0)
 			(effects
@@
 			(project "GamesMachine"
 				(path "/8b2932eb-08c7-412c-8772-7207c8d67aa1"
-					(reference "S5c")
+					(reference "S5c1")
 					(unit 1)
 				)
@@
 		(on_board yes)
 		(dnp no)
-		(property "Reference" "S6c"
+		(property "Reference" "S6c1"
 			(at 187.49 335.61 0)
 			(effects
@@
 			(project "GamesMachine"
 				(path "/8b2932eb-08c7-412c-8772-7207c8d67aa1"
-					(reference "S6c")
+					(reference "S6c1")
 					(unit 1)
 				)
@@
 		(on_board yes)
 		(dnp no)
-		(property "Reference" "S3a"
+		(property "Reference" "S3a1"
 			(at 126.72 317.37 0)
 			(effects
@@
 			(project "GamesMachine"
 				(path "/8b2932eb-08c7-412c-8772-7207c8d67aa1"
-					(reference "S3a")
+					(reference "S3a1")
 					(unit 1)
 				)
@@
 		(on_board yes)
 		(dnp no)
-		(property "Reference" "S4b"
+		(property "Reference" "S4b1"
 			(at 513.79 156.31 0)
 			(effects
@@
 			(project "GamesMachine"
 				(path "/8b2932eb-08c7-412c-8772-7207c8d67aa1"
-					(reference "S4b")
+					(reference "S4b1")
 					(unit 1)
 				)
@@
 		(on_board yes)
 		(dnp no)
-		(property "Reference" "UNITS"
+		(property "Reference" "UNITS1"
 			(at 297.18 339.598 0)
 			(effects
@@
 			(project "GamesMachine"
 				(path "/8b2932eb-08c7-412c-8772-7207c8d67aa1"
-					(reference "UNITS")
+					(reference "UNITS1")
 					(unit 1)
 				)
@@
 		(on_board yes)
 		(dnp no)
-		(property "Reference" "S4a"
+		(property "Reference" "S4a1"
 			(at 126.72 337.37 0)
 			(effects
@@
 			(project "GamesMachine"
 				(path "/8b2932eb-08c7-412c-8772-7207c8d67aa1"
-					(reference "S4a")
+					(reference "S4a1")
 					(unit 1)
 				)
@@
 		(on_board yes)
 		(dnp no)
-		(property "Reference" "S5a"
+		(property "Reference" "S5a1"
 			(at 126.72 357.37 0)
 			(effects
@@
 			(project "GamesMachine"
 				(path "/8b2932eb-08c7-412c-8772-7207c8d67aa1"
-					(reference "S5a")
+					(reference "S5a1")
 					(unit 1)
 				)
@@
 		(on_board yes)
 		(dnp no)
-		(property "Reference" "PWR"
+		(property "Reference" "PWR1"
 			(at 371 277.75 0)
 			(effects
@@
 			(project "GamesMachine"
 				(path "/8b2932eb-08c7-412c-8772-7207c8d67aa1"
-					(reference "PWR")
+					(reference "PWR1")
 					(unit 1)
 				)
@@
 		(on_board yes)
 		(dnp no)
-		(property "Reference" "S6d"
+		(property "Reference" "S6d1"
 			(at 237.49 365.61 0)
 			(effects
@@
 			(project "GamesMachine"
 				(path "/8b2932eb-08c7-412c-8772-7207c8d67aa1"
-					(reference "S6d")
+					(reference "S6d1")
 					(unit 1)
 				)
@@
 		(on_board yes)
 		(dnp no)
-		(property "Reference" "TENS"
+		(property "Reference" "TENS1"
 			(at 367.03 339.042 0)
 			(effects
@@
 			(project "GamesMachine"
 				(path "/8b2932eb-08c7-412c-8772-7207c8d67aa1"
-					(reference "TENS")
+					(reference "TENS1")
 					(unit 1)
 				)
@@
 		(on_board yes)
 		(dnp no)
-		(property "Reference" "S5b"
+		(property "Reference" "S5b1"
 			(at 513.79 176.31 0)
 			(effects
@@
 			(project "GamesMachine"
 				(path "/8b2932eb-08c7-412c-8772-7207c8d67aa1"
-					(reference "S5b")
+					(reference "S5b1")
 					(unit 1)
 				)
@@
 		(on_board yes)
 		(dnp no)
-		(property "Reference" "S6a"
+		(property "Reference" "S6a1"
 			(at 126.72 377.37 0)
 			(effects
@@
 			(project "GamesMachine"
 				(path "/8b2932eb-08c7-412c-8772-7207c8d67aa1"
-					(reference "S6a")
+					(reference "S6a1")
 					(unit 1)
 				)
@@
 		(on_board yes)
 		(dnp no)
-		(property "Reference" "S3b"
+		(property "Reference" "S3b1"
 			(at 513.79 136.31 0)
 			(effects
@@
 			(project "GamesMachine"
 				(path "/8b2932eb-08c7-412c-8772-7207c8d67aa1"
-					(reference "S3b")
+					(reference "S3b1")
 					(unit 1)
 				)
