File: GamesMachine.kicad_pcb (KiCad board)
At the start: 2 copper layers, 160 x 90 mm, 84 parts, among them IC1 7413, IC10 7480, IC11 7412, IC2 7472, IC3 7490, IC4 7490, IC5 7447, IC6 7447, IC9 7425

Commit message: Apply LOGIC_0 -> GND net merge to PCB
Ran Update PCB from Schematic in Pcbnew so the board file picks up the
LOGIC_0 -> GND rename from d471d4e. LOGIC_0 no longer appears anywhere
in the PCB; the previously floating pads (IC2 pins 3/4/5, IC3 and IC4
pins 6/7) now sit on /GND.

Routing and zone fill still need checking in Pcbnew before this is
fabrication-ready.
Parts:
- renumbered PWR to PWR1, S3a to S3a1, S3b to S3b1, S4a to S4a1, S4b to S4b1, S5a to S5a1, S5b to S5b1, S5c to S5c1, S6a to S6a1, S6b to S6b1, S6c to S6c1, S6d to S6d1, TENS to TENS1, UNITS to UNITS1
Connections:
- IC1 pad 7: /GND -> /+5V
- IC2 pad 3: /LOGIC_0 -> /GND
- IC2 pad 4: /LOGIC_0 -> /GND
- IC2 pad 5: /LOGIC_0 -> /GND
- IC3 pad 6: /LOGIC_0 -> /GND
- IC3 pad 7: /LOGIC_0 -> /GND
- IC4 pad 6: /LOGIC_0 -> /GND
- IC4 pad 7: /LOGIC_0 -> /GND
- S3a1 pad 3: /LOGIC_0 -> /GND
- S3b1 pad 3: /LOGIC_0 -> /GND
- S5a1 pad 3: /LOGIC_0 -> /GND
- S6c1 pad 2: /LOGIC_0 -> /GND
- S6d1 pad 2: /LOGIC_0 -> /GND
Routing:
- net /LOGIC_0: track 177.5 -> 0.00 mm
- net /GND: track 292.2 -> 399.8 mm
- net /IC2_CLR: track 195.6 -> 165.8 mm, vias 3 -> 2
- net /LOGIC_1: track 291.2 -> 316.6 mm, vias 1 -> 2
- net /IC3_QC: track 148.7 -> 128.3 mm, vias 2 -> 1
- net /IC4_QB: track 122.1 -> 106.0 mm, vias 2 -> 3
- net /+5V: track 338.5 -> 323.9 mm, vias 3 -> 2
- net /S6B_DICE_TENS7: track 52.3 -> 40.9 mm, vias 0 -> 1
- net /N_TR3C: track 107.6 -> 116.7 mm
- net /TENS_DISP_C: track 47.1 -> 39.9 mm
- net /N_TR2C: track 97.0 -> 90.0 mm
- net /N_TR1E: track 80.8 -> 87.7 mm
- net /UNITS_DISP_E: track 58.8 -> 65.3 mm, vias 0 -> 1
- net /N_TR3B: track 97.1 -> 103.5 mm
- net /IC3_QB: track 132.4 -> 138.7 mm, vias 1 -> 0
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- removed copper zone on B.Cu, net /GND
- removed copper zone on F.Cu, net /GND

Commit message: Rotate all 17 diodes 180 degrees to restore routing geometry
Follow-on to the diode symbol pin-number fix. After that change the pad
numbering swapped but the parts stayed put, which inverted the layout:
the common decode bus landed on the row the individual counter traces
used to occupy and vice versa, making the area awkward to route.

Rotating each diode 180 degrees puts pad 1 where pad 2 physically sat,
so the net at every physical pad location is identical to rev 1.0 again
and the original routing topology works -- while pad 1, which carries
the silkscreen cathode band, is now the electrical cathode. That is the
actual defect being fixed.

KiCad rotates a footprint about pad 1 rather than its centre, so each
origin was moved onto pad 2's former absolute position to cancel the
sideways shift. Footprint child elements (properties, silk text, pads)
carry absolute angles, so those were advanced 180 degrees to stay in
step; Z1's pads needed an explicit 180 added since they carried no angle
at its former 0 degree placement.

Verified against the rev 1.0 board in 9736491: net at each physical pad
position is unchanged, pad numbers are flipped at those positions, and
DRC reports 0 violations.
Parts:
- moved Z1 10.2 mm to (162.0, 88.0), turned to 180 degrees
- moved D10 7.62 mm to (82.8, 88.7), turned to 270 degrees
- moved D11 7.62 mm to (87.2, 88.7), turned to 270 degrees
- moved D12 7.62 mm to (91.7, 88.7), turned to 270 degrees
- moved D13 7.62 mm to (96.2, 88.7), turned to 270 degrees
- moved D14 7.62 mm to (100.7, 88.7), turned to 270 degrees
- moved D15 7.62 mm to (105.1, 88.7), turned to 270 degrees
- moved D16 7.62 mm to (109.6, 88.7), turned to 270 degrees
- moved D17 7.62 mm to (114.1, 88.7), turned to 270 degrees
- moved D18 7.62 mm to (118.6, 88.7), turned to 270 degrees
- moved D19 7.62 mm to (123.0, 88.7), turned to 270 degrees
- moved D20 7.62 mm to (127.5, 88.7), turned to 270 degrees
- moved D5 7.62 mm to (60.4, 88.7), turned to 270 degrees
- moved D6 7.62 mm to (64.9, 88.7), turned to 270 degrees
- moved D7 7.62 mm to (69.4, 88.7), turned to 270 degrees
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Connections:
- D10 pad 1: /S5B_POOLS64 -> /IC3_QC
- D10 pad 2: /IC3_QC -> /S5B_POOLS64
- D11 pad 1: /S4A_ROULETTE37 -> /IC3_QA
- D11 pad 2: /IC3_QA -> /S4A_ROULETTE37
- D12 pad 1: /S4A_ROULETTE37 -> /IC3_QB
- D12 pad 2: /IC3_QB -> /S4A_ROULETTE37
- D13 pad 1: /S4A_ROULETTE37 -> /IC4_QA
- D13 pad 2: /IC4_QA -> /S4A_ROULETTE37
- D14 pad 1: /S4A_ROULETTE37 -> /IC4_QB
- D14 pad 2: /IC4_QB -> /S4A_ROULETTE37
- D15 pad 1: /S4A_ROULETTE37 -> /IC4_QC
- D15 pad 2: /IC4_QC -> /S4A_ROULETTE37
- D16 pad 1: /S4B_ROULETTE44 -> /IC4_QC
- D16 pad 2: /IC4_QC -> /S4B_ROULETTE44
- D17 pad 1: /S4B_ROULETTE44 -> /IC3_QC
- D17 pad 2: /IC3_QC -> /S4B_ROULETTE44
- D18 pad 1: /S6B_DICE_TENS7 -> /IC3_QA
- D18 pad 2: /IC3_QA -> /S6B_DICE_TENS7
- D19 pad 1: /S6B_DICE_TENS7 -> /IC3_QB
- D19 pad 2: /IC3_QB -> /S6B_DICE_TENS7
- D20 pad 1: /S6B_DICE_TENS7 -> /IC3_QC
- D20 pad 2: /IC3_QC -> /S6B_DICE_TENS7
- D5 pad 1: /S6A_DICE_UNITS7 -> /IC4_QA
- D5 pad 2: /IC4_QA -> /S6A_DICE_UNITS7
- D6 pad 1: /S6A_DICE_UNITS7 -> /IC4_QB
- D6 pad 2: /IC4_QB -> /S6A_DICE_UNITS7
- D7 pad 1: /S6A_DICE_UNITS7 -> /IC4_QC
- D7 pad 2: /IC4_QC -> /S6A_DICE_UNITS7
- D8 pad 1: /S5B_POOLS64 -> /IC4_QC
- D8 pad 2: /IC4_QC -> /S5B_POOLS64
- D9 pad 1: /S5B_POOLS64 -> /IC3_QB
- D9 pad 2: /IC3_QB -> /S5B_POOLS64
- Z1 pad 1: /GND -> /+5V
- Z1 pad 2: /+5V -> /GND
Routing:
- net /GND: track 399.8 -> 0.00 mm, vias 2 -> 0
- net /+5V: track 323.9 -> 0.00 mm, vias 2 -> 0
- net /LOGIC_1: track 316.6 -> 0.00 mm, vias 2 -> 0
- net /IC2_CLR: track 165.8 -> 0.00 mm, vias 2 -> 0
- net /+17V: track 154.2 -> 0.00 mm, vias 1 -> 0
- net /IC3_QB: track 138.7 -> 0.00 mm
- net /IC3_QC: track 128.3 -> 0.00 mm, vias 1 -> 0
- net /IC4_QA: track 121.4 -> 0.00 mm, vias 2 -> 0
- net /IC4_QC: track 117.1 -> 0.00 mm, vias 1 -> 0
- net /N_TR3C: track 116.7 -> 0.00 mm, vias 1 -> 0
- net /IC3_QA: track 112.1 -> 0.00 mm, vias 1 -> 0
- net /CLK_B1: track 111.6 -> 0.00 mm
- net /S6A_DICE_UNITS7: track 108.7 -> 0.00 mm, vias 1 -> 0
- net /IC4_QB: track 106.0 -> 0.00 mm, vias 3 -> 0
- net /N_TR3B: track 103.5 -> 0.00 mm, vias 1 -> 0
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
Commit message: Re-route board after diode pad swap and rotation
Full re-route in Pcbnew following the diode polarity fix. 793 segments,
DRC clean: 0 violations, 0 unconnected items.
Connections:
- TR1 pad 2: /N_TR12_BASE -> unconnected-(TR1-C-Pad2)
- TR1 pad 3: unconnected-(TR1-C-Pad3) -> /N_TR12_BASE
- TR2 pad 2: /N_TR12_BASE -> /N_TR2C
- TR2 pad 3: /N_TR2C -> /N_TR12_BASE
- TR3 pad 2: /N_TR3B -> /N_TR3C
- TR3 pad 3: /N_TR3C -> /N_TR3B
Routing:
- net /GND: track 0.00 -> 371.1 mm, vias 0 -> 3
- net /+5V: track 0.00 -> 316.7 mm, vias 0 -> 2
- net /LOGIC_1: track 0.00 -> 297.2 mm, vias 0 -> 1
- net /IC2_CLR: track 0.00 -> 171.0 mm, vias 0 -> 2
- net /+17V: track 0.00 -> 150.8 mm, vias 0 -> 1
- net /IC3_QC: track 0.00 -> 140.9 mm, vias 0 -> 1
- net /IC3_QB: track 0.00 -> 133.5 mm, vias 0 -> 2
- net /IC4_QA: track 0.00 -> 132.8 mm, vias 0 -> 2
- net /IC4_QC: track 0.00 -> 121.6 mm
- net /N_TR3C: track 0.00 -> 111.8 mm, vias 0 -> 1
- net /CLK_B1: track 0.00 -> 111.8 mm, vias 0 -> 2
- net /S6A_DICE_UNITS7: track 0.00 -> 107.3 mm, vias 0 -> 1
- net /IC3_QA: track 0.00 -> 106.9 mm, vias 0 -> 2
- net /N_TR3B: track 0.00 -> 101.6 mm, vias 0 -> 1
- net /IC4_QB: track 0.00 -> 100.7 mm, vias 0 -> 1
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
Commit message: Swap UNITS and TENS display positions
The two displays sat in reverse reading order: UNITS on the left at
x=149, TENS on the right at x=164, so every result read with its digits
transposed (the board showed 41 for the value 14). Wiring and silkscreen
were self-consistent, so this was purely a placement problem -- but it
masqueraded as a Roulette range failure during bring-up.

Exchanged the two footprint placements. Both are identical DIP-14
footprints at the same Y with no rotation, so this is a straight swap of
their (at ...) positions, and each display keeps its own segment nets.

Segment resistor banks left in place: R11-R17 and R18-R24 are horizontal
rows already spanning the full width above both displays, so only the
routing between them changes.

Display area now needs re-routing -- DRC reports 14 shorts and 14
unconnected, since the old copper stayed put while the footprints moved.
Parts:
- moved TENS1 15.0 mm to (149.0, 63.8)
- moved UNITS1 15.0 mm to (164.0, 63.8)
Changed lines of the file:
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@@
 	(footprint "Package_DIP:DIP-14_W7.62mm"
 		(layer "F.Cu")
-		(at 164 63.84)
+		(at 149 63.84)
 		(descr "14-lead though-hole mounted DIP package, row spacing 7.62mm (300 mils)")
 		(tags "THT DIP DIL PDIP 2.54mm 7.62mm 300mil")
@@
 	(footprint "Package_DIP:DIP-14_W7.62mm"
 		(layer "F.Cu")
-		(at 149 63.84)
+		(at 164 63.84)
 		(descr "14-lead though-hole mounted DIP package, row spacing 7.62mm (300 mils)")
 		(tags "THT DIP DIL PDIP 2.54mm 7.62mm 300mil")

Commit message: Re-route display area and TR1-TR3 after placement and pin-order fixes
Re-routed following the UNITS/TENS display swap and the 2N2926 pin-order
correction. 789 segments, 0 unconnected items.

Two starved_thermal errors remain, both on former LOGIC_0 pads that now
belong to GND (IC3 pad 7 and S5a1 pad 3): each reaches only an isolated
island of the top-layer pour rather than the main zone. Both pads are
plated-through and the GND zone is present on both layers, so they are
very likely still solidly grounded via the bottom zone -- rev 1.0
shipped with one warning of this same class. Cleanest fixes are a track
from IC3 pad 7 to IC3 pad 10 (the rev 1.0 bodge wire, in copper) and a
stitching via beside S5a1 pad 3.
Routing:
- net /IC4_QA: track 132.8 -> 160.3 mm, vias 2 -> 1
- net /TENS_DISP_B: track 45.8 -> 23.0 mm, vias 1 -> 0
- net /TENS_G: track 89.3 -> 107.5 mm, vias 0 -> 1
- net /UNITS_DISP_A: track 34.9 -> 51.2 mm, vias 0 -> 1
- net /UNITS_DISP_C: track 44.1 -> 59.8 mm, vias 0 -> 1
- net /TENS_DISP_G: track 27.3 -> 42.7 mm, vias 0 -> 1
- net /TENS_DISP_F: track 23.3 -> 38.3 mm, vias 0 -> 1
- net /UNITS_DISP_B: track 45.4 -> 58.8 mm, vias 0 -> 1
- net /UNITS_DISP_F: track 47.4 -> 35.7 mm, vias 1 -> 0
- net /TENS_DISP_A: track 30.9 -> 19.4 mm, vias 1 -> 0
- net /TENS_DISP_C: track 41.2 -> 29.8 mm, vias 1 -> 0
- net /UNITS_DISP_G: track 51.0 -> 40.4 mm
- net /UNITS_DISP_E: track 58.7 -> 48.3 mm, vias 1 -> 0
- net /TENS_DISP_D: track 45.2 -> 34.8 mm, vias 1 -> 0
- net /IC3_QB: track 133.5 -> 123.2 mm
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- added copper zone on B.Cu, net /GND
- added copper zone on F.Cu, net /GND

Commit message: Add stitching vias to clear the two starved thermal warnings
IC3 pad 7 and S5a1 pad 3 -- both former LOGIC_0 pads now on GND -- each
reached only an isolated island of the top-layer pour rather than the
main zone.

Added a short 0.5 mm stub from each pad to a 0.6/0.3 mm via down to the
bottom ground zone, matching the board's existing track and via sizes.
The stub is deliberate: it makes the connection independent of which
fragment of the pour the via lands in. Nearest non-ground copper is
about 1 mm from each via.

DRC now reports 0 violations and 0 unconnected, though the zone fill in
the file predates the vias -- needs a re-pour in Pcbnew to confirm.
Routing:
- net /GND: track 374.7 -> 376.7 mm, vias 0 -> 2
Changed lines of the file:
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@@
 	)
 	(embedded_fonts no)
+	(segment
+		(start 96.0617 66.1779)
+		(end 97.001 66.52)
+		(width 0.5)
+		(layer "F.Cu")
+		(net 1)
+	)
+	(via
+		(at 97.001 66.52)
+		(size 0.6)
+		(drill 0.3)
+		(layers "F.Cu" "B.Cu")
+		(net 1)
+	)
+	(segment
+		(start 99.0 105.9864)
+		(end 98.0 105.986)
+		(width 0.5)
+		(layer "F.Cu")
+		(net 1)
+	)
+	(via
+		(at 98.0 105.986)
+		(size 0.6)
+		(drill 0.3)
+		(layers "F.Cu" "B.Cu")
+		(net 1)
+	)
 )
